Commit message: feat(ridgeback): static ridgeback ur10e works for grasping

File: mani_skill/assets/robots/ridgeback_ur10e/ridgeback_ur10e.urdf (robot description, URDF)
Before this commit: robot ridgebackur10e, 53 links, 52 joints
Joints:
- joint theta: limit effort=10000 velocity=1.5708 -> lower=-6.283185307179586 upper=6.283185307179586 effort=330.0 velocity=2.0943951023931953; type continuous -> revolute

Commit message: feat(mobile base): working with constraining the motion and point cloud

File: mani_skill/assets/robots/ridgeback_ur10e/ridgeback_ur10e.urdf (robot description, URDF)
Before this commit: robot ridgebackur10e, 53 links, 52 joints
Joints:
- joint theta: limit lower=-6.283185307179586 upper=6.283185307179586 effort=330.0 velocity=2.0943951023931953 -> lower=-1.585 upper=3.5 effort=330.0 velocity=2.0943951023931953
