Commit message: pick block

File: mani_skill/assets/robots/ridgeback_ur10e/static_ridgeback_ur10e.urdf (robot description, URDF)
Before this commit: robot ridgebackur10e, 51 links, 50 joints
Joints:
- joint ur_arm_shoulder_pan_joint: limit lower=-6.283185307179586 upper=6.283185307179586 effort=330.0 velocity=2.0943951023931953 -> lower=-0.78 upper=3.8 effort=330.0 velocity=2.0943951023931953
